Commit message: new urdf

File: reachy2_mujoco/description/original_urdf/reachy2.urdf (robot description, URDF)
Before this commit: robot reachy2, 78 links, 77 joints
Links:
- removed link back_bar
- removed link left_bar
- removed link logo
- removed link right_bar
- removed link sr_cam_l_frame
- removed link sr_cam_l_optical
- removed link sr_cam_r_frame
- removed link sr_cam_r_optical
- removed link world
- added link antenna_left_link, mass 0.001; visual mesh filename=reachy_description/meshes/head_antenna_visual.dae
- added link antenna_right_link, mass 0.001; visual mesh filename=reachy_description/meshes/head_antenna_visual.dae
- added link back_bar_base, mass 0.759; collision box size=0.05 0.05 0.485; visual box size=0.04 0.04 0.485
- added link back_bar_inner, mass 0.759; collision box size=0.05 0.05 0.485; visual box size=0.03 0.03 0.485
- added link depth_cam_l_frame, mass 0.001
- added link depth_cam_l_optical, mass 0.001
- added link depth_cam_r_frame, mass 0.001
- added link depth_cam_r_optical, mass 0.001
- added link depth_cam_rgb_frame, mass 0.001
- added link depth_cam_rgb_optical, mass 0.001
- added link drivewhl1_extra_link
- added link drivewhl1_link, mass 0.5; collision cylinder length=0.035 radius=0.105
- added link drivewhl2_extra_link
- added link drivewhl2_link, mass 0.5; collision cylinder length=0.035 radius=0.105
- added link drivewhl3_extra_link
- added link drivewhl3_link, mass 0.5; collision cylinder length=0.035 radius=0.105
- added link l_arm_tip_bottom, mass 0.001
- added link left_bar_anchor, mass 1.759; collision box size=0.03 0.03 0.03; visual box size=0.03 0.03 0.03
- added link left_bar_base, mass 1.759; collision box size=0.05 0.05 0.485; visual box size=0.04 0.04 0.485
- added link left_bar_inner, mass 0.759; collision box size=0.05 0.05 0.485; visual box size=0.03 0.03 0.485
- added link lidar_link, mass 0.125; collision cylinder length=0.055 radius=0.0508
- added link r_arm_tip_bottom, mass 0.001
- added link right_bar_anchor, mass 1.759; collision box size=0.03 0.03 0.03; visual box size=0.03 0.03 0.03
- added link right_bar_base, mass 1.759; collision box size=0.05 0.05 0.485; visual box size=0.04 0.04 0.485
- added link right_bar_inner, mass 0.759; collision box size=0.05 0.05 0.485; visual box size=0.03 0.03 0.485
- added link tof_camera, mass 1e-5
- added link tof_camera_optical
- link base_link: geometry collision cylinder length=0.19 radius=0.245; visual mesh filename=reachy_description/meshes/mobile_base_visual.dae
- link l_elbow_arm_link: geometry collision mesh filename=reachy_description/meshes/upper_arm_collider.dae; visual mesh filename=reachy_description/meshes/upper_arm_visual.dae
- link l_elbow_first_link: geometry visual mesh filename=orbita2d_description/meshes/2D_sphere_visual.dae
- link l_elbow_forearm_link: geometry collision mesh filename=reachy_description/meshes/forearm_collider.dae; visual mesh filename=reachy_description/meshes/forearm_visual.dae
- link l_hand_distal_link: geometry collision mesh filename=dynamixel_description/meshes/pincette_distal_collider.dae; visual mesh filename=dynamixel_description/meshes/pincette_distal.dae
- link l_hand_distal_mimic_link: geometry collision mesh filename=dynamixel_description/meshes/pincette_distal_collider.dae; visual mesh filename=dynamixel_description/meshes/pincette_distal.dae
- link l_hand_palm_link: geometry collision mesh filename=dynamixel_description/meshes/pincette_base_collider.dae; visual mesh filename=dynamixel_description/meshes/pincette_base_visual.dae
- link l_hand_proximal_link: geometry collision mesh filename=dynamixel_description/meshes/pincette_proximal_collider.dae; visual mesh filename=dynamixel_description/meshes/pincette_proximal_visual.dae
- link l_hand_proximal_mimic_link: geometry collision mesh filename=dynamixel_description/meshes/pincette_proximal_collider.dae; visual mesh filename=dynamixel_description/meshes/pincette_proximal_visual.dae
- link l_hand_virtual_gripper_link: mass 0.001 -> 0.01
- link l_shoulder_first_link: geometry visual mesh filename=orbita2d_description/meshes/2D_sphere_visual.dae
- link l_wrist_link: geometry 
- link r_elbow_arm_link: geometry collision mesh filename=reachy_description/meshes/upper_arm_collider.dae; visual mesh filename=reachy_description/meshes/upper_arm_visual.dae
- link r_elbow_first_link: geometry visual mesh filename=orbita2d_description/meshes/2D_sphere_visual.dae
- link r_elbow_forearm_link: geometry collision mesh filename=reachy_description/meshes/forearm_collider.dae; visual mesh filename=reachy_description/meshes/forearm_visual.dae
- link r_hand_distal_link: geometry collision mesh filename=file:///home/reachy/reachy_ws/install/dynamixel_description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; visual mesh filename=file:///home/reachy/reachy_ws/install/dynamixel_description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
- link r_hand_distal_mimic_link: geometry collision mesh filename=file:///home/reachy/reachy_ws/install/dynamixel_description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; visual mesh filename=file:///home/reachy/reachy_ws/install/dynamixel_description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
- link r_hand_palm_link: geometry collision mesh filename=file:///home/reachy/reachy_ws/install/dynamixel_description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; visual mesh filename=file:///home/reachy/reachy_ws/install/dynamixel_description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
- link r_hand_proximal_link: geometry collision mesh filename=file:///home/reachy/reachy_ws/install/dynamixel_description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; visual mesh filename=file:///home/reachy/reachy_ws/install/dynamixel_description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
- link r_hand_proximal_mimic_link: geometry collision mesh filename=file:///home/reachy/reachy_ws/install/dynamixel_description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; visual mesh filename=file:///home/reachy/reachy_ws/install/dynamixel_description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
- link r_hand_virtual_gripper_link: mass 0.001 -> 0.01
- link r_shoulder_first_link: geometry visual mesh filename=orbita2d_description/meshes/2D_sphere_visual.dae
- link r_wrist_link: geometry 
- link torso: geometry collision mesh filename=reachy_description/meshes/torso_collider.dae; visual mesh filename=reachy_description/meshes/torso_visual.dae
Joints:
- removed joint left_bar_joint
- removed joint logo_joint
- removed joint right_bar_joint
- removed joint sr_cam_l_frame_joint
- removed joint sr_cam_l_optical_joint
- removed joint sr_cam_r_frame_joint
- removed joint sr_cam_r_optical_joint
- removed joint world_joint
- added joint antenna_left: type revolute, parent head, child antenna_left_link, origin xyz=-0.023 0.055 0.091 rpy=0.07374016089676041 -1.061282358260192 -1.0035643198967394, axis 0 0 1, limit lower=-1.5707963267948966 upper=1.5707963267948966 effort=0.0 velocity=0.0
- added joint antenna_right: type revolute, parent head, child antenna_right_link, origin xyz=-0.023 -0.055 0.091 rpy=-0.07374016089676041 -1.061282358260192 1.0035643198967394, axis 0 0 1, limit lower=-1.5707963267948966 upper=1.5707963267948966 effort=0.0 velocity=0.0
- added joint depth_cam_l_frame_joint: type fixed, parent torso, child depth_cam_l_frame, origin xyz=0.058 0.025 -0.03 rpy=0.0 0.8290313946973066 0.0
- added joint depth_cam_l_optical_joint: type fixed, parent torso, child depth_cam_l_optical, origin xyz=0.058 0.025 -0.03 rpy=-2.399827721492203 0.0 -1.5707963267948966
- added joint depth_cam_r_frame_joint: type fixed, parent torso, child depth_cam_r_frame, origin xyz=0.058 -0.025 -0.03 rpy=0.0 0.8290313946973066 0.0 
- added joint depth_cam_r_optical_joint: type fixed, parent torso, child depth_cam_r_optical, origin xyz=0.058 -0.025 -0.03 rpy=-2.399827721492203 0.0 -1.5707963267948966
- added joint depth_cam_rgb_frame_joint: type fixed, parent torso, child depth_cam_rgb_frame, origin xyz=0.058 0.0155 -0.03 rpy=0.0 0.8290313946973066 0.0
- added joint depth_cam_rgb_optical_joint: type fixed, parent torso, child depth_cam_rgb_optical, origin xyz=0.058 0.0155 -0.03 rpy=-2.399827721492203 0.0 -1.5707963267948966
- added joint drivewhl1_extra_joint: type fixed, parent drivewhl1_link, child drivewhl1_extra_link, origin xyz=0 0 0 rpy=0 0 0, axis 0 0 0
- added joint drivewhl1_joint: type fixed, parent base_link, child drivewhl1_link, origin xyz=0.09900000000000003 -0.17147302994931884 0.105 rpy=0 0 0.5235987755982989, axis 0 1 0
- added joint drivewhl2_extra_joint: type fixed, parent drivewhl2_link, child drivewhl2_extra_link, origin xyz=0 0 0 rpy=0 0 0, axis 0 0 0
- added joint drivewhl2_joint: type fixed, parent base_link, child drivewhl2_link, origin xyz=0.09900000000000003 0.17147302994931884 0.105 rpy=0 0 -3.6651914291880923, axis 0 1 0
- added joint drivewhl3_extra_joint: type fixed, parent drivewhl3_link, child drivewhl3_extra_link, origin xyz=0 0 0 rpy=0 0 0, axis 0 0 0
- added joint drivewhl3_joint: type fixed, parent base_link, child drivewhl3_link, origin xyz=-0.198 -2.4248006623117595e-17 0.105 rpy=0 0 -1.5707963267948966, axis 0 1 0
- added joint l_tip_joint_bottom: type fixed, parent l_hand_palm_link, child l_arm_tip_bottom, origin xyz=-0.028 0 0.14432 rpy=3.141592653589793 0 0
- added joint left_bar_anchor_to_base: type fixed, parent base_link, child left_bar_anchor, origin xyz=0.084 0.066 0.241 rpy=0 0 0
- added joint left_bar_joint_mimic: type revolute, parent torso, child left_bar_inner, origin xyz=0 0.048 -0.258 rpy=0 0 0.19088666029061982, axis 0 1 0, limit lower=-1.0 upper=1.0 effort=0.01 velocity=0.01, mimic joint=tripod_joint multiplier=0.2864183599287582 offset=-0.1967146343049915
- added joint left_bar_prism_joint_mimic: type prismatic, parent left_bar_inner, child left_bar_base, origin xyz=0 0 -0.485 rpy=0 0 0, axis 0 0 1, limit lower=-1.0 upper=1.0 effort=1.0 velocity=0.5, mimic joint=tripod_joint multiplier=-0.9861535348976198 offset=0.4814718126556904
- added joint lidar_joint: type fixed, parent base_link, child lidar_link, origin xyz=0.184 0 0.25 rpy=0 0 3.141592653589793
- added joint r_tip_joint_bottom: type fixed, parent r_hand_palm_link, child r_arm_tip_bottom, origin xyz=-0.028 0 0.14432 rpy=3.141592653589793 0 0
- added joint right_bar_anchor_to_base: type fixed, parent base_link, child right_bar_anchor, origin xyz=0.084 -0.066 0.241 rpy=0 0 0
- added joint right_bar_joint_mimic: type revolute, parent torso, child right_bar_inner, origin xyz=0 -0.048 -0.258 rpy=0 0 -0.19088666029061982, axis 0 1 0, limit lower=-1.0 upper=1.0 effort=0.01 velocity=0.01, mimic joint=tripod_joint multiplier=0.2864183599287582 offset=-0.1967146343049915
- added joint right_bar_prism_joint_mimic: type prismatic, parent right_bar_inner, child right_bar_base, origin xyz=0 0 -0.485 rpy=0 0 0, axis 0 0 1, limit lower=-1.0 upper=1.0 effort=1.0 velocity=0.5, mimic joint=tripod_joint multiplier=-0.9861535348976198 offset=0.4814718126556904
- added joint tof_cam_fixed: type fixed, parent head, child tof_camera, origin xyz=0.05643 0 0.061954 rpy=0.0 0.0 0
- added joint tof_camera_optical_joint: type fixed, parent tof_camera, child tof_camera_optical, origin xyz=0 0 0 rpy=-1.5707963267948966 0 -1.5707963267948966
- added joint tripod_joint: type prismatic, parent back_bar_base, child back_bar_inner, origin xyz=0 0 0.035 rpy=0 0 0, axis 0 0 1, limit lower=0.0 upper=0.210 effort=1.0 velocity=0.1
- joint back_bar_joint: child back_bar -> back_bar_base; origin xyz=-0.122 0 0.164 rpy=0 0 0 -> xyz=-0.09 0 0.241 rpy=0 0 0
- joint head_tip_fixed: origin xyz=0.057 0.0 0.056 rpy=0 0.0 0 -> xyz=0.05643 0.0 0.062 rpy=0 0.0 0
- joint l_elbow_yaw: limit lower=-1.5707963267948966 upper=1.5707963267948966 effort=1000.0 velocity=100.0 -> lower=-3.141592653589793 upper=3.141592653589793 effort=1000.0 velocity=100.0
- joint l_hand_finger_proximal_mimic: origin xyz=-0.010196 -0.03792 0.070028 rpy=0 0 3.141592 -> xyz=-0.010196 -0.03792 0.070028 rpy=0 0 3.141592653589793
- joint l_shoulder_base_joint: origin xyz=0.0 0.2 0.0 rpy=-1.7453292519943295 0 -0.2617993877991494 -> xyz=0.0 0.2 0.0 rpy=-1.3089969389957472 0 -0.17453292519943295
- joint l_shoulder_pitch: limit lower=-1.5707963267948966 upper=1.5707963267948966 effort=1000.0 velocity=100.0 -> lower=-3.141592653589793 upper=3.141592653589793 effort=1000.0 velocity=100.0
- joint l_shoulder_roll: limit lower=-0.0 upper=1.5707963267948966 effort=1000.0 velocity=100.0 -> lower=-0.0 upper=3.141592653589793 effort=1000.0 velocity=100.0
- joint l_tip_joint: origin xyz=0 0 0.1 rpy=3.141592653589793 0 0 -> xyz=0.0 0 0.10 rpy=3.141592653589793 0 0
- joint l_wrist_base_joint: origin xyz=0 0 0.28 rpy=3.141592653589793 0 1.5707963267948966 -> xyz=0 0 0.28 rpy=3.141592 0 1.5707963267948966
- joint l_wrist_pitch: limit lower=-0.7853981633974483 upper=0.7853981633974483 effort=1000.0 velocity=100.0 -> lower=-0.35 upper=0.35 effort=1000.0 velocity=100.0
- joint l_wrist_roll: limit lower=-0.7853981633974483 upper=0.7853981633974483 effort=1000.0 velocity=100.0 -> lower=-0.35 upper=0.35 effort=1000.0 velocity=100.0
- joint left_cam_fixed: origin xyz=0.03531 0.0325 0.056 rpy=0.0 0.0  -0.0 -> xyz=0.03531 0.0325 0.062 rpy=0.0 0.0  -0.0
- joint neck_base_joint: origin xyz=0.0 0 0.125 rpy=0 0.17453292519943295 0.0 -> xyz=0.0 0 0.115 rpy=0 0.17453292519943295 0.0
- joint r_elbow_yaw: limit lower=-1.5707963267948966 upper=1.5707963267948966 effort=1000.0 velocity=100.0 -> lower=-3.141592653589793 upper=3.141592653589793 effort=1000.0 velocity=100.0
- joint r_hand_finger_proximal_mimic: origin xyz=-0.010196 -0.03792 0.070028 rpy=0 0 3.141592 -> xyz=-0.010196 -0.03792 0.070028 rpy=0 0 3.141592653589793
- joint r_shoulder_base_joint: origin xyz=0.0 -0.2 0.0 rpy=1.7453292519943295 0 0.2617993877991494 -> xyz=0.0 -0.2 0.0 rpy=1.3089969389957472 0 0.17453292519943295
- joint r_shoulder_pitch: limit lower=-1.5707963267948966 upper=1.5707963267948966 effort=1000.0 velocity=100.0 -> lower=-3.141592653589793 upper=3.141592653589793 effort=1000.0 velocity=100.0
- joint r_shoulder_roll: limit lower=-1.5707963267948966 upper=0.0 effort=1000.0 velocity=100.0 -> lower=-3.141592653589793 upper=0.0 effort=1000.0 velocity=100.0
- joint r_tip_joint: origin xyz=0 0 0.1 rpy=3.141592653589793 0 0 -> xyz=0.0 0 0.10 rpy=3.141592653589793 0 0
- joint r_wrist_base_joint: origin xyz=0 0 0.28 rpy=3.141592653589793 0 1.5707963267948966 -> xyz=0 0 0.28 rpy=3.141592 0 1.5707963267948966
- joint r_wrist_pitch: limit lower=-0.7853981633974483 upper=0.7853981633974483 effort=1000.0 velocity=100.0 -> lower=-0.35 upper=0.35 effort=1000.0 velocity=100.0
- joint r_wrist_roll: limit lower=-0.7853981633974483 upper=0.7853981633974483 effort=1000.0 velocity=100.0 -> lower=-0.35 upper=0.35 effort=1000.0 velocity=100.0
- joint right_cam_fixed: origin xyz=0.03531 -0.0325 0.056 rpy=0.0 0.0 0.0 -> xyz=0.03531 -0.0325 0.062 rpy=0.0 0.0 0.0
- joint torso_base: origin xyz=0.0768 0 0.8360000000000001 rpy=0 0 0 -> xyz=0.08 0 0.72 rpy=0 0 0; parent back_bar -> back_bar_inner

Commit message: change camera to work with updated mujoco plugin (neck link issue)

File: reachy2_mujoco/description/modified_urdf/reachy2.urdf (robot description, URDF)
Before this commit: robot reachy2, 78 links, 77 joints
Links:
- removed link left_camera_optical
- removed link right_camera_optical
- removed link sr_cam_r_optical
- added link left_camera_optical_frame, mass 0.001
- added link right_camera_optical_frame
- added link sr_cam_r_optical_frame, mass 0.001
Joints:
- joint left_camera_optical_joint: child left_camera_optical -> left_camera_optical_frame
- joint right_camera_optical_joint: child right_camera_optical -> right_camera_optical_frame
- joint sr_cam_r_optical_joint: child sr_cam_r_optical -> sr_cam_r_optical_frame

Commit message: save state

File: reachy2_mujoco/description/modified_urdf/reachy2.urdf (robot description, URDF)
Before this commit: robot reachy2, 96 links, 95 joints
Links:
- added link depth_cam_optical_frame, mass 0.001
- added link left_camera_optical_frame, mass 0.001
Joints:
- added joint depth_cam_optical_frame_joint: type fixed, parent torso, child depth_cam_optical_frame, origin xyz=0.058 0.0155 -0.03 rpy=-2.399827721492203 0.0 -1.5707963267948966
- added joint left_camera_optical_frame_joint: type fixed, parent left_camera, child left_camera_optical_frame, origin xyz=0 0 0 rpy=-1.5707963267948966 0 -1.5707963267948966
